Commit message: Update for dec 2023 session

File: TP-DRL/urdf/RoboticArm_2DOF_2.urdf (robot description, URDF)
Before this commit: robot RobotArm_2DOF, 5 links, 4 joints
Links:
- link base_link: geometry collision box size=0.3 0.3 0.02; visual box size=0.3 0.3 0.02
Joints:
- joint Revolute1: limit lower=0. upper=3.1416 -> lower=0. upper=3.1416 effort=5000 velocity=6
- joint Revolute2: limit lower=-3.1416 upper=3.1416 -> lower=-3.1416 upper=3.1416 effort=5000 velocity=6

Commit message: Update for dec 2023 session

File: TP-DRL/urdf/RoboticArm_2DOF_2.urdf (robot description, URDF)
Before this commit: robot RobotArm_2DOF, 5 links, 4 joints
Links:
- link base_link: geometry visual box size=0.3 0.3 0.02
Joints:
- joint Revolute1: limit lower=0. upper=3.1416 effort=5000 velocity=6 -> lower=0. upper=3.1416
- joint Revolute2: limit lower=-3.1416 upper=3.1416 effort=5000 velocity=6 -> lower=-3.1416 upper=3.1416
